File: kicad/lcd_breakout.sch (KiCad schematic (older format))
At the start: 4 parts, among them J1 Conn_01x05_Male, U1 AY0438X-P, U2 DE119

Commit message: Work on routing
Parts:
- J1: footprint Connector_PinHeader_2.54mm:PinHeader_1x05_P2.54mm_Vertical_SMD_Pin1Right -> Connector_PinHeader_2.54mm:PinHeader_1x05_P2.54mm_Vertical
Connections:
- net GND: now also C1.1; no longer C1.2
- net at U1.31 (LCD0): now also C1.2; no longer C1.1
- net VCC renamed VDD
- no-connect marks 0 -> 7
Changed lines of the file:
@@
-$EndComp
-$Comp
-L power:VCC #PWR04
-U 1 1 5EA9E564
-P 4450 1300
-F 0 "#PWR04" H 4450 1150 50  0001 C CNN
-F 1 "VCC" H 4467 1473 50  0000 C CNN
-F 2 "" H 4450 1300 50  0001 C CNN
-F 3 "" H 4450 1300 50  0001 C CNN
-	1    4450 1300
-	1    0    0    -1
 $EndComp
 $Comp
@@
 Wire Wire Line
 	4450 5550 4450 5700
-Wire Wire Line
-	4450 1300 4450 1650
 $Comp
 L power:GND #PWR02
@@
 	1    0    0    -1
 $EndComp
-$Comp
-L power:VCC #PWR01
-U 1 1 5EAA0A11
-P 2500 1750
-F 0 "#PWR01" H 2500 1600 50  0001 C CNN
-F 1 "VCC" H 2517 1923 50  0000 C CNN
-F 2 "" H 2500 1750 50  0001 C CNN
-F 3 "" H 2500 1750 50  0001 C CNN
-	1    2500 1750
-	1    0    0    -1
-$EndComp
 Wire Wire Line
 	2050 1850 3850 1850
@@
 F 3 "~" H 3200 2600 50  0001 C CNN
 	1    3200 2600
-	1    0    0    -1
+	-1   0    0    1
 $EndComp
 Wire Wire Line
 	3200 2450 3850 2450
-$Comp
-L power:GND #PWR03
-U 1 1 5EAA297E
-P 3200 2800
-F 0 "#PWR03" H 3200 2550 50  0001 C CNN
-F 1 "GND" H 3205 2627 50  0000 C CNN
-F 2 "" H 3200 2800 50  0001 C CNN
-F 3 "" H 3200 2800 50  0001 C CNN
-	1    3200 2800
-	1    0    0    -1
-$EndComp
-Wire Wire Line
-	3200 2750 3200 2800
 $Comp
 L lcd_breakout:DE119 U2
@@
 F 0 "J1" H 1956 2328 50  0000 C CNN
 F 1 "Conn_01x05_Male" H 1956 2237 50  0000 C CNN
-F 2 "Connector_PinHeader_2.54mm:PinHeader_1x05_P2.54mm_Vertical_SMD_Pin1Right" H 1850 1950 50  0001 C CNN
+F 2 "Connector_PinHeader_2.54mm:PinHeader_1x05_P2.54mm_Vertical" H 1850 1950 50  0001 C CNN
 F 3 "~" H 1850 1950 50  0001 C CNN
 	1    1850 1950
@@
 Wire Wire Line
 	2050 2150 2500 2150
-Wire Wire Line
-	2050 1750 2500 1750
+NoConn ~ 6700 3000
+NoConn ~ 6700 3100
+NoConn ~ 6700 3200
+NoConn ~ 6700 3300
+NoConn ~ 6700 3400
+NoConn ~ 6700 3500
+NoConn ~ 5050 1850
+$Comp
+L power:GND #PWR0105
+U 1 1 5EB53FF8
+P 3200 3050
+F 0 "#PWR0105" H 3200 2800 50  0001 C CNN
+F 1 "GND" H 3205 2877 50  0000 C CNN
+F 2 "" H 3200 3050 50  0001 C CNN
+F 3 "" H 3200 3050 50  0001 C CNN
+	1    3200 3050
+	1    0    0    -1
+$EndComp
+Wire Wire Line
+	3200 2750 3200 2900
+$Comp
+L power:GND #PWR0106
+U 1 1 5EB551E0
+P 3400 3050
+F 0 "#PWR0106" H 3400 2800 50  0001 C CNN
+F 1 "GND" H 3405 2877 50  0000 C CNN
+F 2 "" H 3400 3050 50  0001 C CNN
+F 3 "" H 3400 3050 50  0001 C CNN
+	1    3400 3050
+	1    0    0    -1
+$EndComp
+Wire Wire Line
+	3200 2900 3400 2900
+Wire Wire Line
+	3400 2900 3400 3050
+Connection ~ 3200 2900
+Wire Wire Line
+	3200 2900 3200 3050
+$Comp
+L power:VDD #PWR0101
+U 1 1 5EB5712D
+P 4250 1400
+F 0 "#PWR0101" H 4250 1250 50  0001 C CNN
+F 1 "VDD" H 4267 1573 50  0000 C CNN
+F 2 "" H 4250 1400 50  0001 C CNN
+F 3 "" H 4250 1400 50  0001 C CNN
+	1    4250 1400
+	1    0    0    -1
+$EndComp
+Wire Wire Line
+	4250 1400 4450 1400
+Wire Wire Line
+	4450 1400 4450 1650
+$Comp
+L power:VDD #PWR0102
+U 1 1 5EB59991
+P 2700 1700
+F 0 "#PWR0102" H 2700 1550 50  0001 C CNN
+F 1 "VDD" H 2717 1873 50  0000 C CNN
+F 2 "" H 2700 1700 50  0001 C CNN
+F 3 "" H 2700 1700 50  0001 C CNN
+	1    2700 1700
+	1    0    0    -1
+$EndComp
+Wire Wire Line
+	2700 1750 2700 1700
+Wire Wire Line
+	2050 1750 2700 1750
 $EndSCHEMATC

Commit message: update images and small clean up
Changed lines of the file:
@@
 encoding utf-8
 Sheet 1 1
-Title ""
-Date ""
-Rev ""
-Comp ""
+Title "LCD Breakout Board"
+Date "2020-05-10"
+Rev "v1.0"
+Comp "Tarn Barford"
 Comment1 ""
 Comment2 ""
@@
 	1    0    0    -1
 $EndComp
-Wire Wire Line
-	3200 2750 3200 2900
-$Comp
-L power:GND #PWR0106
-U 1 1 5EB551E0
-P 3400 3050
-F 0 "#PWR0106" H 3400 2800 50  0001 C CNN
-F 1 "GND" H 3405 2877 50  0000 C CNN
-F 2 "" H 3400 3050 50  0001 C CNN
-F 3 "" H 3400 3050 50  0001 C CNN
-	1    3400 3050
-	1    0    0    -1
-$EndComp
-Wire Wire Line
-	3200 2900 3400 2900
-Wire Wire Line
-	3400 2900 3400 3050
-Connection ~ 3200 2900
-Wire Wire Line
-	3200 2900 3200 3050
 $Comp
 L power:VDD #PWR0101
@@
 Wire Wire Line
 	2050 1750 2700 1750
+Wire Wire Line
+	3200 2750 3200 3050
 $EndSCHEMATC
